File: white_24V/led_ring.kicad_pcb (KiCad board)
At the start: 2 copper layers, 36 x 36 mm, 26 parts, among them J1 Conn_01x02, M1 MOUNT_HOLE_4-40, M2 MOUNT_HOLE_4-40, M3 MOUNT_HOLE_4-40, M4 MOUNT_HOLE_4-40

Commit message: Finished initial design.
Parts:
- R1, R2, R3: value 49.9 -> 402
Other:
- board text added: "24V"
- board text added: "Ring Light 17mm ID, 1 Row, 18 LED (white) Dickinson Lab 2021"
- board text removed: "9V"
- board text removed: "Ring Light 17mm ID, 1 Row, 18 LED Dickinson Lab 2021"
