File: white_24V/led_ring.sch (KiCad schematic (older format))
At the start: 22 parts, among them J1 Conn_01x02

Commit message: Finished initial design.
Parts:
- R1, R2, R3: value 49.9 -> 402
Other:
- note added: "24V"
- note added: "LED: white 20mA max, Vf = 3V\nManufacturer: Foshan NationStar Optoelectronics NCD0805W2 \nLCSC: C84258\n"
- note removed: "LED: 940nm 65mA max, Vf = 1.2V\nmanufacturer: Everlight Elec IR17-21C/TR8, \nLCSC: C131250\n"
Changed lines of the file:
@@
 	1    0    0    -1
 $EndComp
-Text Notes 4100 3050 0    60   ~ 0
-LED:   940nm  65mA max,  Vf = 1.2V\nmanufacturer:  Everlight Elec  IR17-21C/TR8,   \nLCSC: C131250\n
+Text Notes 3750 3150 0    60   ~ 0
+LED:   white  20mA max,  Vf = 3V\nManufacturer:   Foshan NationStar Optoelectronics  NCD0805W2 \nLCSC: C84258\n
 $Comp
 L power:PWR_FLAG #FLG03
@@
 P 6200 1900
 F 0 "R1" V 5993 1900 50  0000 C CNN
-F 1 "49.9" V 6084 1900 50  0000 C CNN
+F 1 "402" V 6084 1900 50  0000 C CNN
 F 2 "Resistor_SMD:R_0805_2012Metric" V 6130 1900 50  0001 C CNN
 F 3 "~" H 6200 1900 50  0001 C CNN
@@
 P 6200 2350
 F 0 "R2" V 5993 2350 50  0000 C CNN
-F 1 "49.9" V 6084 2350 50  0000 C CNN
+F 1 "402" V 6084 2350 50  0000 C CNN
 F 2 "Resistor_SMD:R_0805_2012Metric" V 6130 2350 50  0001 C CNN
 F 3 "~" H 6200 2350 50  0001 C CNN
@@
 P 6200 1450
 F 0 "R3" V 5993 1450 50  0000 C CNN
-F 1 "49.9" V 6084 1450 50  0000 C CNN
+F 1 "402" V 6084 1450 50  0000 C CNN
 F 2 "Resistor_SMD:R_0805_2012Metric" V 6130 1450 50  0001 C CNN
 F 3 "~" H 6200 1450 50  0001 C CNN
@@
 	6700 1450 6700 1900
 Connection ~ 6700 1900
+Text Notes 2810 2385 0    50   ~ 0
+24V
 $EndSCHEMATC
